File: LED-Matrix-PCB/LED-Matrix-PCB.kicad_pcb (KiCad board)
At the start: 2 copper layers, 25 parts, among them J1 Raspberry_Pi_2_3, J2 Barrel_Jack, J3 SW1, J4 LED_Matrix, J5 SW2, J6 SW3, J7 Joystick, J8 SW4, J9 POWER

Commit message: Complete
Parts:
- J1: footprint LED-Matrix-PCB:raspberrypi_2_3 -> Connector_PinHeader_2.54mm:PinHeader_2x20_P2.54mm_Vertical; moved to B.Cu
- moved J7 94.7 mm to (108.2, 83.1), turned to 0 degrees
- moved J2 82.9 mm to (111.3, 90.2)
- moved J3 78.8 mm to (124.7, 83.1)
- moved J5 73.3 mm to (133.9, 83.1)
- moved LED_Matrix 66.4 mm to (123.7, 99.1), turned to 90 degrees
- moved J8 62.9 mm to (151.6, 83.1)
- moved J6 61.6 mm to (142.7, 83.1)
- moved Matrix_POWER 48.5 mm to (151.4, 100.3)
- moved R6 39.2 mm to (120.1, 90.8)
- moved R8 31.6 mm to (141.7, 90.9), turned to 180 degrees
- moved R4 30.8 mm to (120.1, 87.6)
- moved R5 30.3 mm to (124.7, 87.6)
- moved C3 27.5 mm to (141.7, 87.6)
- moved C7 24.3 mm to (106.7, 87.6)
- moved C2 23.4 mm to (133.6, 87.6)
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- renumbered J4 to LED_Matrix, J9 to Matrix_POWER
Routing:
- net GPIO16: track 0.00 -> 98.3 mm, vias 0 -> 3
- net GPIO26: track 0.00 -> 77.4 mm
- net GND: track 0.00 -> 77.2 mm, vias 0 -> 8
- net +5V: track 0.00 -> 64.3 mm
- net GPIO2: track 0.00 -> 63.5 mm
- net +3V3: track 0.00 -> 57.8 mm
- net GPIO3: track 0.00 -> 57.2 mm
- net GPIO5: track 0.00 -> 51.2 mm
- net GPIO4: track 0.00 -> 46.6 mm
- net GPIO6: track 0.00 -> 38.5 mm
- net GPIO27: track 0.00 -> 33.2 mm
- net GPIO12: track 0.00 -> 29.4 mm
- net GPIO17: track 0.00 -> 29.0 mm
- net GPIO23: track 0.00 -> 28.9 mm
- net GPIO7: track 0.00 -> 27.7 mm, vias 0 -> 1
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- added copper zone on B.Cu, net GND
Other:
- board outline added: 55.1 x 36 mm
- board text added: "16x32-LED-Matrix"
- board text added: "Made By kyh github.com/1q2f3d"
