File: LED-Matrix-PCB/LED-Matrix-PCB.sch (KiCad schematic (older format))
At the start: 24 parts

Commit message: Update LED-Matrix-PCB.sch
Parts:
- added J9: POWER, Connector_Molex:Molex_SPOX_5267-02A_1x02_P2.50mm_Vertical, symbol Connector_Generic:Conn_01x02
- gave numbers to parts that had none: 24
Connections:
- net +5V: now also J9.1 (Pin_1)
- net GND: now also J9.2 (Pin_2)
Other:
- moved on the sheet: J2

Commit message: Complete
Parts:
- J1: footprint LED-Matrix-PCB:raspberrypi_2_3 -> Connector_PinHeader_2.54mm:PinHeader_2x20_P2.54mm_Vertical
Changed lines of the file:
@@
 F 0 "J1" H 2550 5281 50  0000 C CNN
 F 1 "Raspberry_Pi_2_3" H 2550 5190 50  0000 C CNN
-F 2 "LED-Matrix-PCB:raspberrypi_2_3" H 2550 3800 50  0001 C CNN
+F 2 "Connector_PinHeader_2.54mm:PinHeader_2x20_P2.54mm_Vertical" H 2550 3800 50  0001 C CNN
 F 3 "https://www.raspberrypi.org/documentation/hardware/raspberrypi/schematics/rpi_SCH_3bplus_1p0_reduced.pdf" H 2550 3800 50  0001 C CNN
 	1    2550 3800
